File: Input_Switch_8X.kicad_sch (KiCad schematic)
At the start: 6 parts

Commit message: dev1
Parts:
- H1, H2, H3, H4: renamed from U; value (none) -> MountingHole_Pad; footprint (none) -> MountingHole:MountingHole_3.2mm_M3_Pad_Via
- J10: renamed from J; value Conn_01x04 -> GND; footprint (none) -> Connector_PinHeader_2.54mm:PinHeader_2x02_P2.54mm_Vertical
- J9: renamed from J; value Conn_01x04 -> VCC; footprint (none) -> Connector_PinHeader_2.54mm:PinHeader_2x02_P2.54mm_Vertical
