File: Switch_LED.kicad_sch (KiCad schematic)
At the start: 10 parts

Commit message: dev1
Parts:
- D1: renamed from D; footprint (none) -> LED_SMD:LED_0603_1608Metric
- D2: renamed from D; value D_Zener_Small -> BZT52C10; footprint (none) -> Library:D_SOD-123
- J1: renamed from J; footprint (none) -> Library:PinHeader_1x02_P2.54mm_Vertical
- R1: renamed from R; value R_Small -> 33R; footprint (none) -> Resistor_SMD:R_0603_1608Metric
- R5: renamed from R; value R_Small -> 1k; footprint (none) -> Resistor_SMD:R_0603_1608Metric
- R6: renamed from R; value R_Small -> 10k; footprint (none) -> Resistor_SMD:R_0603_1608Metric
- SW1: renamed from SW; footprint (none) -> Library:SW_PUSH_6mm_H5mm
- SW2: renamed from SW; footprint (none) -> Library:SW_Toggle_Blue_wSlots_2_Pins
- renumbered Q to Q1, Q to Q2
